Commit message: Update envimo.urdf

File: URDF/envimo.urdf (robot description, URDF)
Before this commit: robot envimo, 8 links, 7 joints
Links:
- added link camera0_link; collision box size=0.09 0.025 0.025; visual box size=0.09 0.025 0.025
Joints:
- removed joint frontLefttWheel_frontAxel_joint
- removed joint rearLefttWheel_rearAxel_joint
- added joint camera0_base_joint: type fixed, parent base_link, child camera0_link, origin xyz=0.3426 0 0.0134 rpy=0 0 0
- added joint frontLeftWheel_frontAxel_joint: type continuous, parent frontAxel_link, child frontLeftWheel_link, origin xyz=0.0 0.26 -0.055 rpy=0 0 0, axis 0 1 0
- added joint rearLeftWheel_rearAxel_joint: type continuous, parent rearAxel_link, child rearLeftWheel_link, origin xyz=0.0 0.26 -0.055 rpy=0 0 0, axis 0 1 0
- joint frontAxel_base_joint: limit lower=-.5 upper=.5 effort=5 velocity=1.0 -> lower=-0.5 upper=0.5 effort=5 velocity=1.0; origin xyz=0.24 0 -0.275 rpy=0.0 0.0 0.0 -> xyz=0.24 0 -0.275 rpy=0 0 0
- joint frontRightWheel_frontAxel_joint: axis 00 1 0 -> 0 1 0; origin xyz=0.0 -0.26 -0.055 rpy=0 0.0 0.0 -> xyz=0.0 -0.26 -0.055 rpy=0 0 0
- joint rearAxel_link_base_joint: origin xyz=-0.24 0 -0.275 rpy=0.0 0.0 0.0 -> xyz=-0.24 0 -0.275 rpy=0 0 0
- joint rearRightWheel_rearAxel_joint: axis 00 1 0 -> 0 1 0; origin xyz=0.0 -0.26 -0.055 rpy=0 0.0 0.0 -> xyz=0.0 -0.26 -0.055 rpy=0 0 0
- joint world_base_joint: origin xyz=2 1 0.0 rpy=0.0 0.0 0.0 -> xyz=2 1 0.4316 rpy=0 0 0

Commit message: add camera and inertia 28 kg

File: URDF/envimo.urdf (robot description, URDF)
Before this commit: robot envimo, 9 links, 8 joints
Links:
- link base_link: mass None -> 28.0

Commit message: add base footprint

File: URDF/envimo.urdf (robot description, URDF)
Before this commit: robot envimo, 9 links, 8 joints
Links:
- removed link world_link
- added link base_footprint
Joints:
- removed joint world_base_joint
- added joint base_footprint_joint: type fixed, parent base_link, child base_footprint, origin xyz=0 0 0 rpy=0 0 0
