Commit message: Update envimo_all_joints_fixed.urdf

File: URDF/envimo_all_joints_fixed.urdf (robot description, URDF)
Before this commit: robot envimo, 9 links, 8 joints
Links:
- removed link camera0_link
- added link camera_link; collision box size=0.09 0.025 0.025; visual box size=0.09 0.025 0.025
Joints:
- removed joint camera0_base_joint
- added joint camera_base_joint: type fixed, parent base_link, child camera_link, origin xyz=0.3426 0 0.0134 rpy=0 0 0
