Commit message: Update envimo_all_joints_fixed.urdf

File: urdf/envimo_all_joints_fixed.urdf (robot description, URDF)
Before this commit: robot envimo, 9 links, 8 joints
Links:
- added link laser_link; collision cylinder length=0.05 radius=0.05; visual cylinder length=0.03 radius=0.035
Joints:
- added joint laser_camera_joint: type fixed, parent camera_link, child laser_link, origin xyz=-0.035 0 0.20 rpy=0 0 0

Commit message: Update envimo_all_joints_fixed.urdf
chang the parent of laser from camera to base

File: urdf/envimo_all_joints_fixed.urdf (robot description, URDF)
Before this commit: robot envimo, 10 links, 9 joints
Links:
- link laser_link: geometry collision cylinder length=0.03 radius=0.035; visual cylinder length=0.03 radius=0.035
Joints:
- removed joint laser_camera_joint
- added joint laser_base_joint: type fixed, parent base_link, child laser_link, origin xyz=0.3076 0 0.2134 rpy=0 0 0

Commit message: Update envimo_all_joints_fixed.urdf

File: urdf/envimo_all_joints_fixed.urdf (robot description, URDF)
Before this commit: robot envimo, 10 links, 9 joints
Links:
- removed link laser_link
Joints:
- removed joint laser_base_joint
