Commit message: Update envimo_all_joints_fixed_with_laser.urdf

File: urdf/envimo_all_joints_fixed_with_laser.urdf (robot description, URDF)
Before this commit: robot envimo, 10 links, 9 joints
Links:
- added link base_inertial_link, mass 28.0
- link base_link: mass 28.0 -> None
Joints:
- added joint inertial_to_base: type fixed, parent base_inertial_link, child base_link, origin xyz=0 0 0 rpy=0 0 0

Commit message: Update envimo_all_joints_fixed_with_laser.urdf

File: urdf/envimo_all_joints_fixed_with_laser.urdf (robot description, URDF)
Before this commit: robot envimo, 11 links, 10 joints
Links:
- removed link base_inertial_link
- link base_footprint: mass None -> 28.0
Joints:
- removed joint inertial_to_base

Commit message: Update envimo_all_joints_fixed_with_laser.urdf

File: urdf/envimo_all_joints_fixed_with_laser.urdf (robot description, URDF)
Before this commit: robot envimo, 10 links, 9 joints
Joints:
- joint laser_base_joint: origin xyz=0.3076 0 0.2134 rpy=0 0 0 -> xyz=0.3076 0 0.2134 rpy=0 0 3.1416

Commit message: add gps

File: urdf/envimo_all_joints_fixed_with_laser.urdf (robot description, URDF)
Before this commit: robot envimo, 10 links, 9 joints
Links:
- added link gps_link; collision cylinder length=0.01 radius=0.015; visual cylinder length=0.01 radius=0.015
Joints:
- added joint gps_base_joint: type fixed, parent base_link, child gps_link, origin xyz=0.3076 -0.10 0.2134 rpy=0 0 0

Commit message: add gps and rotate the position

File: urdf/envimo_all_joints_fixed_with_laser.urdf (robot description, URDF)
Before this commit: robot envimo, 11 links, 10 joints
Joints:
- joint gps_base_joint: origin xyz=0.3076 -0.10 0.2134 rpy=0 0 0 -> xyz=0.3 -0.03 0.20 rpy=0 0 -1.5708

Commit message: adding the camera right and left

File: urdf/envimo_all_joints_fixed_with_laser.urdf (robot description, URDF)
Before this commit: robot envimo, 11 links, 10 joints
Links:
- added link camera_left_link; collision box size=0.02 0.02 0.02; visual box size=0.02 0.02 0.02
- added link camera_right_link; collision box size=0.02 0.02 0.02; visual box size=0.02 0.02 0.02
Joints:
- added joint camera_left_base_joint: type fixed, parent base_link, child camera_left_link, origin xyz=0.3426 0.22 0.0134 rpy=0 0 0.7854
- added joint camera_right_base_joint: type fixed, parent base_link, child camera_right_link, origin xyz=0.3426 -0.22 0.0134 rpy=0 0 -0.7854
- joint camera_base_joint: origin xyz=0.3426 0 0.0134 rpy=0 0 0 -> xyz=0.3426 0 0.0134 rpy=0 0.5236 0

Commit message: Update envimo_all_joints_fixed_with_laser.urdf

File: urdf/envimo_all_joints_fixed_with_laser.urdf (robot description, URDF)
Before this commit: robot envimo, 13 links, 12 joints
Links:
- removed link camera_link
- added link center_link; collision box size=0.09 0.025 0.025; visual box size=0.09 0.025 0.025
Joints:
- joint camera_base_joint: child camera_link -> center_link

Commit message: Update envimo_all_joints_fixed_with_laser.urdf

File: urdf/envimo_all_joints_fixed_with_laser.urdf (robot description, URDF)
Before this commit: robot envimo, 13 links, 12 joints
Joints:
- joint camera_base_joint: origin xyz=0.3426 0 0.0134 rpy=0 0.5236 0 -> xyz=0.3426 0 0.0134 rpy=0 0.28 0
- joint camera_left_base_joint: origin xyz=0.3426 0.22 0.0134 rpy=0 0 0.7854 -> xyz=0.3426 0.22 0.0134 rpy=-1.5708 0 -0.7854
- joint camera_right_base_joint: origin xyz=0.3426 -0.22 0.0134 rpy=0 0 -0.7854 -> xyz=0.3426 -0.22 0.0134 rpy=-1.5708 0 -2.3562

Commit message: remove realsense and add third camera instead (camera_center_link)

File: urdf/envimo_all_joints_fixed_with_laser.urdf (robot description, URDF)
Before this commit: robot envimo, 13 links, 12 joints
Links:
- removed link center_link
- added link camera_center_link; collision box size=0.02 0.02 0.02; visual box size=0.02 0.02 0.02
Joints:
- joint camera_base_joint: child center_link -> camera_center_link; origin xyz=0.3426 0 0.0134 rpy=0 0.28 0 -> xyz=0.346 0 0.0134 rpy=0 0 0.2

Commit message: Update envimo_all_joints_fixed_with_laser.urdf

File: urdf/envimo_all_joints_fixed_with_laser.urdf (robot description, URDF)
Before this commit: robot envimo, 13 links, 12 joints
Joints:
- joint camera_base_joint: origin xyz=0.346 0 0.0134 rpy=-1.5708 0 -1.5708 -> xyz=0.346 0 0.0134 rpy=-1.85 0 -1.5708
- joint camera_left_base_joint: origin xyz=0.3426 0.22 0.0134 rpy=-1.5708 0 -0.7854 -> xyz=0.3426 0.22 0.0134 rpy=-1.5708 0 -0.733038
- joint camera_right_base_joint: origin xyz=0.3426 -0.22 0.0134 rpy=-1.5708 0 -2.3562 -> xyz=0.3426 -0.22 0.0134 rpy=-1.5708 0 -2.37365
